Commit message: Adapta Palmares para testes com parametros Oregon

File: description/palmares_bot.urdf.xacro (robot description, xacro)
@@ -4,6 +4,6 @@
     <!-- Include common macros (inertia helpers + materials) -->
     <xacro:include filename="common.xacro"/>
-    <!-- Include lidar (parents to 'chassis' link defined below) -->
-    <xacro:include filename="lidar.xacro"/>
+    <!-- Include Palmares lidar (parents to 'chassis' link defined below) -->
+    <xacro:include filename="palmares_lidar.xacro"/>
     <!-- ══════════════════════════════════════════════════════════════════
          ROBOT DIMENSIONS  (STL in mm → scaled to metres at 0.001)
@@ -14,15 +14,5 @@
          Lidar: Ø36 × H36 mm  at X=0.194 m  Y=0.050 m  Z=0.275 m
     ══════════════════════════════════════════════════════════════════════ -->
-    <!-- ═══ base_footprint (Nav2 ground-level root) ══════════════════════ -->
-    <link name="base_footprint"/>
-    <joint name="base_footprint_joint" type="fixed">
-        <parent link="base_footprint"/>
-        <child link="base_link"/>
-        <origin xyz="0 0 0" rpy="0 0 0"/>
-    </joint>
-    <!-- ═══ base_link (STL body) ══════════════════════════════════════════
-         The STL origin sits at ground level (Z=0).
-         Collision uses the lower half of the body so lidar rays clear freely.
-    ══════════════════════════════════════════════════════════════════════ -->
+    <!-- ═══ base_link (Nav2/Gazebo base frame) ════════════════════════════ -->
     <link name="base_link">
         <visual>
@@ -45,4 +35,11 @@
         </xacro:inertial_box>
     </link>
+    <!-- ═══ base_footprint (ground-level helper frame) ═══════════════════ -->
+    <joint name="base_footprint_joint" type="fixed">
+        <parent link="base_link"/>
+        <child link="base_footprint"/>
+        <origin xyz="0 0 0" rpy="0 0 0"/>
+    </joint>
+    <link name="base_footprint"/>
     <!-- ═══ Wheels ════════════════════════════════════════════════════════
          Wheel centre sits at Z=0.100 m (= wheel radius, exactly at ground).
@@ -131,5 +128,5 @@
     <!-- ═══ Gazebo plugins ════════════════════════════════════════════════ -->
     <gazebo>
-        <!-- Differential Drive: publishes odom + TF odom→base_footprint -->
+        <!-- Differential Drive: publishes odom + TF odom→base_link -->
         <plugin filename="gz-sim-diff-drive-system"
                 name="gz::sim::systems::DiffDrive">
@@ -140,5 +137,5 @@
             <max_linear_acceleration>6.0</max_linear_acceleration>
             <frame_id>odom</frame_id>
-            <child_frame_id>base_footprint</child_frame_id>
+            <child_frame_id>base_link</child_frame_id>
             <tf_topic>/tf</tf_topic>
             <topic>cmd_vel</topic>
