Commit message: Enable simulated camera on Palmares bot

File: description/camera.xacro (robot description, xacro)
@@ -1,26 +1,35 @@
 <?xml version="1.0"?>
 <robot xmlns:xacro="http://www.ros.org/wiki/xacro" >
-    <!-- Camera's urdf -->
+    <!-- Camera's urdf - C720-like (78 deg diagonal FOV, 1280x720 @ 30 fps)
+         Positioned at the same frontal line as the LiDAR (chassis origin X),
+         centred in Y, 4 cm above chassis. -->
     <joint name="camera_joint" type="fixed">
         <parent link="chassis"/>
         <child link="camera_link"/>
-        <origin xyz="0.175 0 0.08" rpy="0 0 0"/>
+        <!-- X: same as lidar (chassis X = 0)
+             Y: -0.075 -> robot frame Y = 0.05 + (-0.075) = -0.025 m (2.5 cm right of centre)
+             Z: 0.09 -> align camera with ArUco marker height -->
+        <origin xyz="0 -0.075 0.09" rpy="0 0 0"/>
     </joint>
     <link name="camera_link">
         <visual>
+            <!-- Approximates a small USB webcam body -->
             <geometry>
-                <box size="0.010 0.03 0.03"/>
+                <box size="0.012 0.075 0.025"/>
             </geometry>
             <material name="black"/>
         </visual>
     </link>
-    <!-- Camera Optical link -->
+    <!-- Standard ROS camera optical frame
+         Rotates from robot convention (X fwd, Y left, Z up)
+         to optical convention (X right, Y down, Z fwd).
+         Required for correct TF2 transforms of ArUco poses. -->
     <joint name="camera_optical_joint" type="fixed">
         <parent link="camera_link"/>
         <child link="camera_link_optical"/>
-        <origin xyz="0 0 0" rpy="0 0 0"/>
+        <origin xyz="0 0 0" rpy="${-pi/2} 0 ${-pi/2}"/>
     </joint>
-    <link name="camera_link_optical"></link>
-    <!-- Camera Gazebo Sensor Plugin -->
+    <link name="camera_link_optical"/>
+    <!-- Camera Gazebo Sensor Plugin - Logitech C720-like -->
     <gazebo reference="camera_link">
         <material>Gazebo/Black</material>
@@ -34,13 +43,14 @@
             <camera>
                 <camera_info_topic>camera/camera_info</camera_info_topic>
-                <horizontal_fov>1.089</horizontal_fov>
+                <!-- C720: ~78 deg diagonal ~= 1.20 rad horizontal FOV at 16:9 -->
+                <horizontal_fov>1.20</horizontal_fov>
                 <image>
                     <format>R8G8B8</format>
-                    <width>640</width>
-                    <height>480</height>
+                    <width>1280</width>
+                    <height>720</height>
                 </image>
                 <clip>
                     <near>0.05</near>
-                    <far>8.0</far>
+                    <far>10.0</far>
                 </clip>
             </camera>

File: description/palmares_bot.urdf.xacro (robot description, xacro)
@@ -3,4 +3,5 @@
     <!-- Robot description for Palmares Bot (differential drive with STL mesh) -->
     <xacro:arg name="tof_lidar" default="true"/>
+    <xacro:arg name="camera" default="true"/>
     <!-- Include common macros (inertia helpers + materials) -->
     <xacro:include filename="common.xacro"/>
@@ -9,4 +10,7 @@
     <xacro:if value="$(arg tof_lidar)">
         <xacro:include filename="palmares_tof_lidar.xacro"/>
+    </xacro:if>
+    <xacro:if value="$(arg camera)">
+        <xacro:include filename="camera.xacro"/>
     </xacro:if>
     <!-- ══════════════════════════════════════════════════════════════════
