Commit message: Update sim spawn and lidar geometry

File: description/palmares_lidar.xacro (robot description, xacro)
@@ -42,5 +42,5 @@
                 </scan>
                 <range>
-                    <min>0.3</min>
+                    <min>0.30</min>
                     <max>12</max>
                 </range>

File: description/palmares_tof_lidar.xacro (robot description, xacro)
@@ -5,10 +5,10 @@
         <parent link="chassis"/>
         <child link="tof_lidar_frame"/>
-        <origin xyz="0.08 0 0.18" rpy="0 0 0"/>
+        <origin xyz="0.065 0 0.18" rpy="0 0 0"/>
     </joint>
     <link name="tof_lidar_frame">
         <visual>
             <geometry>
-                <box size="0.060 0.030 0.030"/>
+                <box size="0.030 0.030 0.030"/>
             </geometry>
             <material name="black"/>
@@ -16,8 +16,8 @@
         <collision>
             <geometry>
-                <box size="0.060 0.030 0.030"/>
+                <box size="0.030 0.030 0.030"/>
             </geometry>
         </collision>
-        <xacro:inertial_box mass="0.05" x="0.060" y="0.030" z="0.030">
+        <xacro:inertial_box mass="0.05" x="0.030" y="0.030" z="0.030">
             <origin xyz="0 0 0" rpy="0 0 0"/>
         </xacro:inertial_box>
